File: Hardware/EagleSchematicv7.sch (EAGLE design)
At the start: 6 parts

Commit message: Add files via upload
Parts:
- removed U$1: NANO, Arduino-clone:NANO
- added JP1, JP2: (no value), adafruit:PINHD-1X18
Connections:
- new net N$6: JP1.10, JP2.2
- net N$1: now also JP2.12; no longer U$1.5.5V
- net N$3: now also JP1.8; no longer U$1.D2
- net N$4: now also JP1.11; no longer U$1.D5
Changed lines of the file:
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@@
 <part name="SW1" library="adafruit" library_urn="urn:adsk.eagle:library:420" deviceset="SWITCH_PUSHBUTTON" device="SOFTTOUCHSMD_SJ" package3d_urn="urn:adsk.eagle:package:6240956/1"/>
 <part name="R2" library="SparkFun-Resistors" library_urn="urn:adsk.eagle:library:532" deviceset="100OHM" device="-0603-1/4W-5%" package3d_urn="urn:adsk.eagle:package:39650/1" value="100"/>
-<part name="U$1" library="Arduino-clone" deviceset="NANO" device=""/>
+<part name="JP1" library="adafruit" library_urn="urn:adsk.eagle:library:420" deviceset="PINHD-1X18" device="" package3d_urn="urn:adsk.eagle:package:6240826/1"/>
+<part name="JP2" library="adafruit" library_urn="urn:adsk.eagle:library:420" deviceset="PINHD-1X18" device="" package3d_urn="urn:adsk.eagle:package:6240826/1"/>
 </parts>
 <sheets>
@@
 <attribute name="VALUE" x="166.624" y="73.66" size="1.778" layer="96" font="vector" rot="R90" align="top-center"/>
 </instance>
-<instance part="U$1" gate="G$1" x="114.3" y="33.02" rot="R180"/>
+<instance part="JP1" gate="A" x="111.76" y="40.64">
+<attribute name="NAME" x="105.41" y="64.135" size="1.778" layer="95"/>
+<attribute name="VALUE" x="105.41" y="12.7" size="1.778" layer="96"/>
+</instance>
+<instance part="JP2" gate="A" x="129.54" y="38.1" rot="R180">
+<attribute name="NAME" x="135.89" y="14.605" size="1.778" layer="95" rot="R180"/>
+<attribute name="VALUE" x="135.89" y="66.04" size="1.778" layer="96" rot="R180"/>
+</instance>
 </instances>
 <busses>
@@
 <wire x1="165.1" y1="78.74" x2="165.1" y2="88.9" width="0.1524" layer="91"/>
 <pinref part="R2" gate="G$1" pin="2"/>
-<pinref part="U$1" gate="G$1" pin="D5"/>
-<wire x1="78.74" y1="35.56" x2="104.14" y2="35.56" width="0.1524" layer="91"/>
+<wire x1="78.74" y1="35.56" x2="109.22" y2="35.56" width="0.1524" layer="91"/>
+<pinref part="JP1" gate="A" pin="11"/>
 </segment>
 </net>
@@
 <wire x1="63.5" y1="78.74" x2="154.94" y2="78.74" width="0.1524" layer="91"/>
 <wire x1="154.94" y1="78.74" x2="154.94" y2="45.72" width="0.1524" layer="91"/>
-<pinref part="U$1" gate="G$1" pin="5.5V"/>
-<wire x1="154.94" y1="45.72" x2="137.16" y2="45.72" width="0.1524" layer="91"/>
+<wire x1="154.94" y1="45.72" x2="132.08" y2="45.72" width="0.1524" layer="91"/>
+<pinref part="JP2" gate="A" pin="12"/>
 </segment>
 </net>
@@
 <wire x1="68.58" y1="33.02" x2="68.58" y2="66.04" width="0.1524" layer="91"/>
 <wire x1="68.58" y1="66.04" x2="91.44" y2="66.04" width="0.1524" layer="91"/>
-<pinref part="U$1" gate="G$1" pin="D2"/>
 <wire x1="91.44" y1="66.04" x2="91.44" y2="43.18" width="0.1524" layer="91"/>
-<wire x1="91.44" y1="43.18" x2="104.14" y2="43.18" width="0.1524" layer="91"/>
+<wire x1="91.44" y1="43.18" x2="109.22" y2="43.18" width="0.1524" layer="91"/>
+<pinref part="JP1" gate="A" pin="8"/>
 </segment>
 </net>
+<net name="N$6" class="0">
+<segment>
+<pinref part="JP1" gate="A" pin="10"/>
+<pinref part="JP2" gate="A" pin="2"/>
+</segment>
+</net>
