File: Electronics/EagleNanov3.brd (EAGLE design)
At the start: 20.3 x 40.3 mm, 7 parts

Commit message: Add files via upload
Connections:
- net GND: now also SW1.P$1; no longer R1.P$2
- net N$1: now also R1.P$2; no longer SW1.P$1
Routing:
- net GND: track 24.2 -> 36.0 mm
- net N$1: track 49.4 -> 38.4 mm
- net N$4: track 4.76 -> 2.96 mm
Changed lines of the file:
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@@
 <vertex x="0" y="0"/>
 </polygon>
-<contactref element="R1" pad="P$2"/>
 <contactref element="LED2" pad="K"/>
-<wire x1="7.62" y1="35.56" x2="7.62" y2="31.75" width="0.508" layer="1"/>
-<wire x1="11.43" y1="27.94" x2="11.43" y2="26.67" width="0.508" layer="1"/>
-<wire x1="7.62" y1="31.75" x2="11.43" y2="27.94" width="0.508" layer="1"/>
-<wire x1="11.43" y1="26.67" x2="11.43" y2="16.51" width="0.508" layer="1"/>
-<wire x1="11.43" y1="16.51" x2="8.89" y2="13.97" width="0.508" layer="1"/>
+<contactref element="SW1" pad="P$1"/>
+<wire x1="11.43" y1="26.67" x2="7.62" y2="30.48" width="0.508" layer="1"/>
+<wire x1="7.62" y1="30.48" x2="7.62" y2="35.56" width="0.508" layer="1"/>
+<wire x1="11.43" y1="26.67" x2="11.43" y2="19.05" width="0.508" layer="1"/>
+<wire x1="6.35" y1="13.97" x2="6.35" y2="3.81" width="0.508" layer="1"/>
+<wire x1="6.35" y1="3.81" x2="6.91" y2="3.81" width="0.508" layer="1"/>
+<wire x1="11.43" y1="19.05" x2="6.35" y2="13.97" width="0.508" layer="1"/>
 </signal>
 <signal name="N$1">
 <contactref element="G1" pad="+"/>
 <contactref element="JP2" pad="15"/>
-<contactref element="SW1" pad="P$1"/>
-<wire x1="12.7" y1="35.56" x2="12.7" y2="33.02" width="0.508" layer="16"/>
-<wire x1="12.7" y1="33.02" x2="15.24" y2="30.48" width="0.508" layer="16"/>
-<wire x1="15.24" y1="30.48" x2="15.24" y2="11.43" width="0.508" layer="16"/>
-<wire x1="15.24" y1="11.43" x2="11.43" y2="7.62" width="0.508" layer="16"/>
-<wire x1="11.43" y1="7.62" x2="5.08" y2="7.62" width="0.508" layer="16"/>
-<wire x1="5.08" y1="7.62" x2="5.08" y2="3.81" width="0.508" layer="16"/>
-<wire x1="5.08" y1="3.81" x2="6.91" y2="3.81" width="0.508" layer="16"/>
 <wire x1="17.78" y1="38.1" x2="13.97" y2="38.1" width="0.508" layer="1"/>
 <wire x1="13.97" y1="38.1" x2="13.97" y2="36.83" width="0.508" layer="1"/>
 <wire x1="13.97" y1="36.83" x2="12.7" y2="35.56" width="0.508" layer="1"/>
+<contactref element="R1" pad="P$2"/>
+<wire x1="12.7" y1="35.56" x2="12.7" y2="31.75" width="0.508" layer="16"/>
+<wire x1="12.7" y1="31.75" x2="15.24" y2="29.21" width="0.508" layer="16"/>
+<wire x1="15.24" y1="29.21" x2="15.24" y2="16.51" width="0.508" layer="16"/>
+<wire x1="15.24" y1="16.51" x2="7.62" y2="16.51" width="0.508" layer="16"/>
+<wire x1="7.62" y1="16.51" x2="7.62" y2="13.97" width="0.508" layer="16"/>
+<wire x1="7.62" y1="13.97" x2="8.89" y2="13.97" width="0.508" layer="16"/>
 </signal>
 <signal name="N$2">
@@
 <contactref element="JP1" pad="8"/>
 <contactref element="R2" pad="1"/>
-<wire x1="6.77" y1="19.05" x2="5.5" y2="20.32" width="0.508" layer="1"/>
 <wire x1="5.5" y1="20.32" x2="2.54" y2="20.32" width="0.508" layer="1"/>
+<wire x1="5.5" y1="20.32" x2="6.77" y2="19.05" width="0" layer="19" extent="1-1"/>
 </signal>
 <signal name="N$5">
 <contactref element="R2" pad="2"/>
 <contactref element="LED2" pad="A"/>
-<wire x1="8.89" y1="26.67" x2="8.47" y2="26.25" width="0.508" layer="1"/>
-<wire x1="8.47" y1="26.25" x2="8.47" y2="19.05" width="0.508" layer="1"/>
+<wire x1="8.47" y1="19.05" x2="8.47" y2="26.25" width="0.508" layer="1"/>
+<wire x1="8.47" y1="26.25" x2="8.89" y2="26.67" width="0.508" layer="1"/>
 </signal>
 </signals>
